Commit message: urdf

File: franka_description/robots/panda_arm_fixed.xacro (robot description, xacro)
@@ -1,5 +1,6 @@
 <?xml version='1.0' encoding='utf-8'?>
 <robot xmlns:xacro="http://www.ros.org/wiki/xacro" name="panda">
-  <xacro:macro name="panda_arm" params="arm_id:='panda' description_pkg:='franka_description' connected_to:='toptop_plate' xyz:='0 0 0.3' rpy:='0 0 0'">
+  <xacro:macro name="panda_arm" params="arm_id:='panda' description_pkg:='franka_description'
+    connected_to:='top_plate' xyz:='-0.05 0 0.05' rpy:='0 0 0'">
     <!-- <xacro:unless value="${not connected_to}">
       <joint name="${arm_id}_joint_${connected_to}" type="fixed">
@@ -38,5 +39,5 @@
       </collision>
     </link>
-    <joint name="${arm_id}_joint1" type="revolute">
+    <joint name="${arm_id}_joint1" type="fixed">
       <safety_controller k_position="100.0" k_velocity="40.0" soft_lower_limit="-2.8973" soft_upper_limit="2.8973"/>
       <origin rpy="0 0 0" xyz="0 0 0.333"/>
@@ -58,5 +59,5 @@
       </collision>
     </link>
-    <joint name="${arm_id}_joint2" type="revolute">
+    <joint name="${arm_id}_joint2" type="fixed">
       <safety_controller k_position="100.0" k_velocity="40.0" soft_lower_limit="-1.7628" soft_upper_limit="1.7628"/>
       <origin rpy="${-pi/2} 0 0" xyz="0 0 0"/>
@@ -78,5 +79,5 @@
       </collision>
     </link>
-    <joint name="${arm_id}_joint3" type="revolute">
+    <joint name="${arm_id}_joint3" type="fixed">
       <safety_controller k_position="100.0" k_velocity="40.0" soft_lower_limit="-2.8973" soft_upper_limit="2.8973"/>
       <origin rpy="${pi/2} 0 0" xyz="0 -0.316 0"/>
@@ -98,5 +99,5 @@
       </collision>
     </link>
-    <joint name="${arm_id}_joint4" type="revolute">
+    <joint name="${arm_id}_joint4" type="fixed">
       <safety_controller k_position="100.0" k_velocity="40.0" soft_lower_limit="-3.0718" soft_upper_limit="0.0175"/>
       <origin rpy="${pi/2} 0 0" xyz="0.0825 0 0"/>
@@ -118,5 +119,5 @@
       </collision>
     </link>
-    <joint name="${arm_id}_joint5" type="revolute">
+    <joint name="${arm_id}_joint5" type="fixed">
       <safety_controller k_position="100.0" k_velocity="40.0" soft_lower_limit="-2.8973" soft_upper_limit="2.8973"/>
       <origin rpy="${-pi/2} 0 0" xyz="-0.0825 0.384 0"/>
@@ -138,5 +139,5 @@
       </collision>
     </link>
-    <joint name="${arm_id}_joint6" type="revolute">
+    <joint name="${arm_id}_joint6" type="fixed">
       <safety_controller k_position="100.0" k_velocity="40.0" soft_lower_limit="-0.0175" soft_upper_limit="3.7525"/>
       <origin rpy="${pi/2} 0 0" xyz="0 0 0"/>
@@ -158,5 +159,5 @@
       </collision>
     </link>
-    <joint name="${arm_id}_joint7" type="revolute">
+    <joint name="${arm_id}_joint7" type="fixed">
       <safety_controller k_position="100.0" k_velocity="40.0" soft_lower_limit="-2.8973" soft_upper_limit="2.8973"/>
       <origin rpy="${pi/2} 0 0" xyz="0.088 0 0"/>
